Commit message: task A.4 complete

File: nuturtle_description/urdf/turtlebot3_burger.urdf.xacro (robot description, xacro)
@@ -3,4 +3,14 @@
   xmlns:xacro="http://ros.org/wiki/xacro">
   <!-- <xacro:include filename="$(find nuturtle_desrciption)/urdf/common_properties.urdf"/> -->
+  <xacro:property name="yaml_file" value="$(find nuturtle_description)/config/diff_params.yaml"/>
+  <xacro:property name="yaml_variables" value="${xacro.load_yaml(yaml_file)['/**']['ros__parameters']}"/>
+  <xacro:property name="wheel_radius" value="${yaml_variables['wheel_radius']}"/>
+  <xacro:property name="track_width" value="${yaml_variables['track_width']}"/>
+  <xacro:property name="motor_cmd_max" value="${yaml_variables['motor_cmd_max']}"/>
+  <xacro:property name="motor_cmd_per_rad_sec" value="${yaml_variables['motor_cmd_per_rad_sec']}"/>
+  <xacro:property name="encoder_ticks_per_rad" value="${yaml_variables['encoder_ticks_per_rad']}"/>
+  <xacro:property name="collision_radius" value="${yaml_variables['collision_radius']}"/>
+  <!-- xacro arguments possible values are red, green, blue, and purple-->
+  <xacro:property name="color" value="$(arg color)"/>
   <!-- Init colour -->
   <material name="black">
@@ -34,4 +44,7 @@
     <color rgba="1.0 1.0 1.0 1.0"/>
   </material>
+  <material name="purple">
+    <color rgba="0.3 0.15 0.52 1.0"/>
+  </material>
   <link name="base_footprint"/>
   <joint name="base_joint" type="fixed">
@@ -46,12 +59,29 @@
         <mesh filename="package://nuturtle_description/meshes/bases/burger_base.stl" scale="0.001 0.001 0.001"/>
       </geometry>
-      <material name="light_black"/>
+        <material name="${color}"/>
+      <!-- <material name="light_black"/> -->
     </visual>
-    <collision>
+    <xacro:if value="${collision_radius &gt; 0.0}">
+      <collision>
+        <origin xyz="-0.032 0 0.070" rpy="0 0 0"/>
+        <geometry>
+          <cylinder length="0.143" radius="${collision_radius}"/>
+        </geometry>
+      </collision>
+    </xacro:if>
+  <xacro:if value="${collision_radius &lt; 0.0}">
+      <collision>
+        <origin xyz="-0.032 0 0.070" rpy="0 0 0"/>
+        <geometry>
+          <box size="0.140 0.140 0.143"/>
+        </geometry>
+      </collision>
+    </xacro:if>
+    <!-- <collision>
       <origin xyz="-0.032 0 0.070" rpy="0 0 0"/>
       <geometry>
         <box size="0.140 0.140 0.143"/>
       </geometry>
-    </collision>
+    </collision> -->
     <inertial>
       <origin xyz="0 0 0" rpy="0 0 0"/>
@@ -77,5 +107,5 @@
       <origin xyz="0 0 0" rpy="0 0 0"/>
       <geometry>
-        <cylinder length="0.018" radius="0.033"/>
+        <cylinder length="0.018" radius="${wheel_radius}"/>
       </geometry>
     </collision>
@@ -103,5 +133,5 @@
       <origin xyz="0 0 0" rpy="0 0 0"/>
       <geometry>
-        <cylinder length="0.018" radius="0.033"/>
+        <cylinder length="0.018" radius="${wheel_radius}"/>
       </geometry>
     </collision>

Commit message: completed yaml file and prefix of task A

File: nuturtle_description/urdf/turtlebot3_burger.urdf.xacro (robot description, xacro)
@@ -93,5 +93,5 @@
     <parent link="base_link"/>
     <child link="wheel_left_link"/>
-    <origin xyz="0.0 0.08 0.023" rpy="-1.57 0 0"/>
+    <origin xyz="0.0 ${track_width/2} 0.023" rpy="-1.57 0 0"/>
     <axis xyz="0 0 1"/>
   </joint>
@@ -119,5 +119,5 @@
     <parent link="base_link"/>
     <child link="wheel_right_link"/>
-    <origin xyz="0.0 -0.080 0.023" rpy="-1.57 0 0"/>
+    <origin xyz="0.0 -${track_width/2} 0.023" rpy="-1.57 0 0"/>
     <axis xyz="0 0 1"/>
   </joint>
